Commit message: link one

File: body.urdf (robot description, URDF)
Before this commit: robot robot, 2 links, 1 joints
Links:
- removed link leg
- added link Leg, mass 1; collision box size=1 1 1; visual box size=1 1 1

Commit message: Working Joints

File: body.urdf (robot description, URDF)
Before this commit: robot robot, 2 links, 1 joints
Links:
- removed link Leg
- added link BackLeg, mass 1; collision box size=1 1 1; visual box size=1 1 1
- added link FrontLeg, mass 1; collision box size=1 1 1; visual box size=1 1 1
Joints:
- removed joint Torso_Leg
- added joint Torso_BackLeg: type revolute, parent Torso, child BackLeg, origin xyz=-0.5 0 1 rpy=0 0 0, axis 0 1 0, limit lower=-3.14159 upper=3.14159 effort=0.0 velocity=0.0
- added joint Torso_FrontLeg: type revolute, parent Torso, child FrontLeg, origin xyz=0.5 0 1 rpy=0 0 0, axis 0 1 0, limit lower=-3.14159 upper=3.14159 effort=0.0 velocity=0.0

Commit message: Deliver 1

File: body.urdf (robot description, URDF)
Before this commit: robot robot, 3 links, 2 joints
Links:
- added link BackFoot, mass 1; collision box size=0.2 0.2 1; visual box size=0.2 0.2 1
- added link FrontFoot, mass 1; collision box size=0.2 0.2 1; visual box size=0.2 0.2 1
- added link LeftFoot, mass 1; collision box size=0.2 0.2 1; visual box size=0.2 0.2 1
- added link LeftLeg, mass 1; collision box size=1 0.2 0.2; visual box size=1 0.2 0.2
- added link RightFoot, mass 1; collision box size=0.2 0.2 1; visual box size=0.2 0.2 1
- added link RightLeg, mass 1; collision box size=1 0.2 0.2; visual box size=1 0.2 0.2
- link BackLeg: geometry collision box size=0.2 1 0.2; visual box size=0.2 1 0.2
- link FrontLeg: geometry collision box size=0.2 1 0.2; visual box size=0.2 1 0.2
Joints:
- added joint BackLeg_BackFoot: type revolute, parent BackLeg, child BackFoot, origin xyz=0 -1 0 rpy=0 0 0, axis 1 0 0, limit lower=-3.14159 upper=3.14159 effort=0.0 velocity=0.0
- added joint FrontLeg_FrontFoot: type revolute, parent FrontLeg, child FrontFoot, origin xyz=0 1 0 rpy=0 0 0, axis 1 0 0, limit lower=-3.14159 upper=3.14159 effort=0.0 velocity=0.0
- added joint LeftLeg_LeftFoot: type revolute, parent LeftLeg, child LeftFoot, origin xyz=1 0 0 rpy=0 0 0, axis 0 1 0, limit lower=-3.14159 upper=3.14159 effort=0.0 velocity=0.0
- added joint RightLeg_RightFoot: type revolute, parent RightLeg, child RightFoot, origin xyz=-1 0 0 rpy=0 0 0, axis 0 1 0, limit lower=-3.14159 upper=3.14159 effort=0.0 velocity=0.0
- added joint Torso_LeftLeg: type revolute, parent Torso, child LeftLeg, origin xyz=0.5 0 1 rpy=0 0 0, axis 0 1 0, limit lower=-3.14159 upper=3.14159 effort=0.0 velocity=0.0
- added joint Torso_RightLeg: type revolute, parent Torso, child RightLeg, origin xyz=-0.5 0 1 rpy=0 0 0, axis 0 1 0, limit lower=-3.14159 upper=3.14159 effort=0.0 velocity=0.0
- joint Torso_BackLeg: axis 0 1 0 -> 1 0 0; origin xyz=-0.5 0 1 rpy=0 0 0 -> xyz=0 -0.5 1 rpy=0 0 0
- joint Torso_FrontLeg: axis 0 1 0 -> 1 0 0; origin xyz=0.5 0 1 rpy=0 0 0 -> xyz=0 0.5 1 rpy=0 0 0

Commit message: B

File: body.urdf (robot description, URDF)
Before this commit: robot robot, 9 links, 8 joints
Links:
- link LeftLeg: geometry collision box size=0.2 1 0.2; visual box size=0.2 1 0.2
- link RightLeg: geometry collision box size=0.2 1 0.2; visual box size=0.2 1 0.2
- link Torso: geometry collision box size=1.5 1 1; visual box size=1.5 1 1
Joints:
- joint LeftLeg_LeftFoot: axis 0 1 0 -> 1 0 0; origin xyz=1 0 0 rpy=0 0 0 -> xyz=0 -1 0 rpy=0 0 0
- joint RightLeg_RightFoot: axis 0 1 0 -> 1 0 0; origin xyz=-1 0 0 rpy=0 0 0 -> xyz=0 1 0 rpy=0 0 0
- joint Torso_LeftLeg: axis 0 1 0 -> 1 0 0; origin xyz=0.5 0 1 rpy=0 0 0 -> xyz=0 -0.5 1 rpy=0 0 0
- joint Torso_RightLeg: axis 0 1 0 -> 1 0 0; origin xyz=-0.5 0 1 rpy=0 0 0 -> xyz=0 0.5 1 rpy=0 0 0
